Commit message: fixing URDF format and frictions

File: rover_description/urdf/materials.xacro (robot description, xacro)
@@ -18,5 +18,5 @@
 # SOFTWARE. -->
 <robot name="materials" xmlns:xacro="http://www.ros.org/wiki/xacro">
-   <material name="red">
+    <material name="red">
         <color rgba="0.8 0 0 1"/>
     </material>

File: rover_description/urdf/sensors/asus_xtion.urdf.xacro (robot description, xacro)
@@ -21,8 +21,8 @@
     <xacro:property name="math_pi_over_2" value="1.5707963267948966" />
     <joint name="${prefix}_joint" type="fixed">
-        <axis xyz="1 0 0"/>
-        <xacro:insert_block name="origin"/>
-        <parent link="${parent}"/>
-        <child link="${prefix}_link"/>
+      <axis xyz="1 0 0"/>
+      <xacro:insert_block name="origin"/>
+      <parent link="${parent}"/>
+      <child link="${prefix}_link"/>
     </joint>
     <link name="${prefix}_link">
@@ -76,5 +76,5 @@
             <far>8.0</far>
           </clip>
-	        <distortion>
+          <distortion>
             <k1>0.00000001</k1>
             <k2>0.00000001</k2>
@@ -137,5 +137,5 @@
                 </publisher>
               </topic>
-             <topic name="/camera/depth/image_raw/theora">
+              <topic name="/camera/depth/image_raw/theora">
                 <publisher>
                   <reliability>best_effort</reliability>

File: rover_description/urdf/sensors/hokuyo.urdf.xacro (robot description, xacro)
@@ -34,5 +34,5 @@
         <origin xyz="0 0 -0.05" rpy="0 0 0"/>
         <geometry>
-            <mesh filename="package://rover_description/meshes/sensors/hokuyo/hokuyo_ust_20lx.dae"/>
+          <mesh filename="package://rover_description/meshes/sensors/hokuyo/hokuyo_ust_20lx.dae"/>
         </geometry>
       </visual>
@@ -44,5 +44,5 @@
     </link>
     <gazebo reference="${prefix}_base_link">
-        <material>Gazebo/DarkGrey</material>
+      <material>Gazebo/DarkGrey</material>
     </gazebo>
     <link name="${prefix}_link">
@@ -54,43 +54,43 @@
     </joint>
     <gazebo reference="${prefix}_link">
-            <sensor type="gpu_ray" name="hokuyo_sensor">
-                <pose>0 0 0 0 0 0</pose>
-                <visualize>true</visualize>
-                <update_rate>50</update_rate>
-                <ray>
-                    <scan>
-                        <horizontal>
-                            <samples>30</samples>
-                            <resolution>1</resolution>
-                            <min_angle>${min_angle}</min_angle>
-                            <max_angle>${max_angle}</max_angle>
-                        </horizontal>
-                    </scan>
-                    <range>
-                        <min>0.06</min>
-                        <max>5.0</max>
-                        <resolution>0.004359297</resolution>
-                    </range>
-                    <noise>
-                        <type>gaussian</type>
-                        <mean>0.0</mean>
-                        <stddev>0.01</stddev>
-                    </noise>
-                </ray>
-                <plugin name="${prefix}_controller" filename="libgazebo_ros_ray_sensor.so">
-                  <ros>
-                    <remapping>~/out:=scan</remapping>
-                    <qos>
-                      <topic name="scan">
-                        <publisher>
-                          <reliability>best_effort</reliability>
-                        </publisher>
-                      </topic>
-                    </qos>
-                  </ros>
-                  <output_type>sensor_msgs/LaserScan</output_type>
-                  <frame_name>${prefix}_link</frame_name>
-                </plugin>
-            </sensor>
+      <sensor type="gpu_ray" name="hokuyo_sensor">
+        <pose>0 0 0 0 0 0</pose>
+        <visualize>true</visualize>
+        <update_rate>50</update_rate>
+        <ray>
+          <scan>
+            <horizontal>
+              <samples>30</samples>
+              <resolution>1</resolution>
+              <min_angle>${min_angle}</min_angle>
+              <max_angle>${max_angle}</max_angle>
+            </horizontal>
+          </scan>
+          <range>
+            <min>0.06</min>
+            <max>5.0</max>
+            <resolution>0.004359297</resolution>
+          </range>
+          <noise>
+            <type>gaussian</type>
+            <mean>0.0</mean>
+            <stddev>0.01</stddev>
+          </noise>
+        </ray>
+        <plugin name="${prefix}_controller" filename="libgazebo_ros_ray_sensor.so">
+          <ros>
+            <remapping>~/out:=scan</remapping>
+            <qos>
+              <topic name="scan">
+                <publisher>
+                  <reliability>best_effort</reliability>
+                </publisher>
+              </topic>
+            </qos>
+          </ros>
+          <output_type>sensor_msgs/LaserScan</output_type>
+          <frame_name>${prefix}_link</frame_name>
+        </plugin>
+      </sensor>
     </gazebo>
   </xacro:macro>

File: rover_description/urdf/sensors/imu.urdf.xacro (robot description, xacro)
@@ -20,8 +20,8 @@
   <xacro:macro name="sensor_imu" params="prefix parent *origin">
     <joint name="${prefix}_joint" type="fixed">
-        <axis xyz="1 0 0"/>
-        <xacro:insert_block name="origin"/>
-        <parent link="${parent}"/>
-        <child link="${prefix}_link"/>
+      <axis xyz="1 0 0"/>
+      <xacro:insert_block name="origin"/>
+      <parent link="${parent}"/>
+      <child link="${prefix}_link"/>
     </joint>
     <link name="${prefix}_link">
@@ -46,5 +46,5 @@
     </link>
     <gazebo reference="${prefix}_link">
-        <material>Gazebo/Blue</material>
+      <material>Gazebo/Blue</material>
     </gazebo>
     <gazebo reference="${prefix}_link">

File: rover_description/urdf/wheels/wheel.urdf.xacro (robot description, xacro)
@@ -46,10 +46,9 @@
         <gazebo reference="${lon_label}_${lat_label}_wheel_link">
             <material>Gazebo/DarkGray</material>
-			<mu1 value="100.0"/>
-			<mu2 value="100.0"/>
-			<kp value="10000000.0" />
-			<kd value="1.0" />
-			<fdir1 value="1 0 0"/>
-            <turnGravityOff>false</turnGravityOff>
+            <mu1>1.0</mu1>
+            <mu2>1.0</mu2>
+            <kp>10000000</kp>
+            <kd>1.0</kd>
+            <fdir1 value="1 0 0"/>
         </gazebo>
     </xacro:macro>
